File: Kicad/v1a/ClockReset.kicad_sch (KiCad schematic)
At the start: 28 parts, among them SW1 RESET

Commit message: Add files relating to v1a and v1b revisions
Parts:
- gave numbers to parts that had none: 15
- renumbered C34 to C1
