File: Kicad/v1a/audio.kicad_sch (KiCad schematic)
At the start: 39 parts, among them U16 74HC139, U17 74HC153, U18 74HC670, U19 74HC670, U20 82C54, U21 82C54 (PLCC), U22 74HC165, U23 74HC165, U24 74HC165, U25 74HC165

Commit message: v1a update
Other:
- note removed: "note: confirm if R/W pinouts are correct"
Changed lines of the file:
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@@
     (stroke (width 0) (type default))
-  )
-  (text "note: confirm if R/W pinouts are correct" (at 26.67 137.16 0)
-    (effects (font (size 1.27 1.27)) (justify left bottom))
   )
   (label "Osc 2" (at 93.98 109.22 0) (fields_autoplaced)

Commit message: Add files relating to v1a and v1b revisions
Parts:
- renumbered R46 to R27, R46 to R36
Changed lines of the file:
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@@
   (symbol (lib_id "Device:R_Small") (at 254 128.27 270) (mirror x) (unit 1)
     (in_bom yes) (on_board yes) (dnp no)
-    (property "Reference" "R46" (at 255.27 127 0)
+    (property "Reference" "R36" (at 255.27 127 0)
       (effects (font (size 1.27 1.27)) (justify left))
     )
@@
     (instances
       (project "v1a"
-        (path "/82bc3382-6295-4121-a2db-2433a00f189b/a5616d11-43a5-47df-90ad-b31b5ddb497a"
-          (reference "R46") (unit 1)
-        )
         (path "/82bc3382-6295-4121-a2db-2433a00f189b/0beb40b4-3ea5-423b-b5b9-637bbdbde287"
           (reference "R36") (unit 1)
@@
   (symbol (lib_id "power:GND") (at 138.43 185.42 270) (unit 1)
     (in_bom yes) (on_board yes) (dnp no) (fields_autoplaced)
-    (property "Reference" "#PWR03" (at 132.08 185.42 0)
+    (property "Reference" "#PWR0107" (at 132.08 185.42 0)
       (effects (font (size 1.27 1.27)) hide)
     )
@@
     (instances
       (project "v1a"
-        (path "/82bc3382-6295-4121-a2db-2433a00f189b"
-          (reference "#PWR03") (unit 1)
-        )
         (path "/82bc3382-6295-4121-a2db-2433a00f189b/0beb40b4-3ea5-423b-b5b9-637bbdbde287"
           (reference "#PWR0107") (unit 1)
@@
   (symbol (lib_id "power:GND") (at 247.65 93.98 180) (unit 1)
     (in_bom yes) (on_board yes) (dnp no)
-    (property "Reference" "#PWR0134" (at 247.65 87.63 0)
+    (property "Reference" "#PWR087" (at 247.65 87.63 0)
       (effects (font (size 1.27 1.27)) hide)
     )
@@
     (instances
       (project "v1a"
-        (path "/82bc3382-6295-4121-a2db-2433a00f189b/a5616d11-43a5-47df-90ad-b31b5ddb497a"
-          (reference "#PWR0134") (unit 1)
-        )
         (path "/82bc3382-6295-4121-a2db-2433a00f189b/0beb40b4-3ea5-423b-b5b9-637bbdbde287"
           (reference "#PWR087") (unit 1)
@@
   (symbol (lib_id "power:GND") (at 29.21 184.15 270) (unit 1)
     (in_bom yes) (on_board yes) (dnp no) (fields_autoplaced)
-    (property "Reference" "#PWR03" (at 22.86 184.15 0)
+    (property "Reference" "#PWR0104" (at 22.86 184.15 0)
       (effects (font (size 1.27 1.27)) hide)
     )
@@
     (instances
       (project "v1a"
-        (path "/82bc3382-6295-4121-a2db-2433a00f189b"
-          (reference "#PWR03") (unit 1)
-        )
         (path "/82bc3382-6295-4121-a2db-2433a00f189b/0beb40b4-3ea5-423b-b5b9-637bbdbde287"
           (reference "#PWR0104") (unit 1)
@@
         (path "/82bc3382-6295-4121-a2db-2433a00f189b/0beb40b4-3ea5-423b-b5b9-637bbdbde287"
           (reference "C4") (unit 1)
-        )
-        (path "/82bc3382-6295-4121-a2db-2433a00f189b/470e69f3-fa8a-41f9-93cf-a95a9c1e6a1d"
-          (reference "C7") (unit 1)
-        )
-        (path "/82bc3382-6295-4121-a2db-2433a00f189b/a5616d11-43a5-47df-90ad-b31b5ddb497a"
-          (reference "C31") (unit 1)
         )
       )
@@
   (symbol (lib_id "Device:R_Small") (at 254 102.87 270) (mirror x) (unit 1)
     (in_bom yes) (on_board yes) (dnp no)
-    (property "Reference" "R46" (at 255.27 100.33 0)
+    (property "Reference" "R27" (at 255.27 100.33 0)
       (effects (font (size 1.27 1.27)) (justify left))
     )
@@
     (instances
       (project "v1a"
-        (path "/82bc3382-6295-4121-a2db-2433a00f189b/a5616d11-43a5-47df-90ad-b31b5ddb497a"
-          (reference "R46") (unit 1)
-        )
         (path "/82bc3382-6295-4121-a2db-2433a00f189b/0beb40b4-3ea5-423b-b5b9-637bbdbde287"
           (reference "R27") (unit 1)
@@
         (path "/82bc3382-6295-4121-a2db-2433a00f189b/0beb40b4-3ea5-423b-b5b9-637bbdbde287"
           (reference "C5") (unit 1)
-        )
-        (path "/82bc3382-6295-4121-a2db-2433a00f189b/470e69f3-fa8a-41f9-93cf-a95a9c1e6a1d"
-          (reference "C7") (unit 1)
-        )
-        (path "/82bc3382-6295-4121-a2db-2433a00f189b/a5616d11-43a5-47df-90ad-b31b5ddb497a"
-          (reference "C31") (unit 1)
         )
       )
@@
   (symbol (lib_id "power:GND") (at 247.65 119.38 180) (unit 1)
     (in_bom yes) (on_board yes) (dnp no)
-    (property "Reference" "#PWR0134" (at 247.65 113.03 0)
+    (property "Reference" "#PWR093" (at 247.65 113.03 0)
       (effects (font (size 1.27 1.27)) hide)
     )
@@
     (instances
       (project "v1a"
-        (path "/82bc3382-6295-4121-a2db-2433a00f189b/a5616d11-43a5-47df-90ad-b31b5ddb497a"
-          (reference "#PWR0134") (unit 1)
-        )
         (path "/82bc3382-6295-4121-a2db-2433a00f189b/0beb40b4-3ea5-423b-b5b9-637bbdbde287"
           (reference "#PWR093") (unit 1)
