File: Kicad/v1a/io.kicad_sch (KiCad schematic)
At the start: 9 parts, among them J1 KeyIN, J2 KeyOUT, U24 74HC138, U25 74HC273, U31 74HCT540

Commit message: Add files relating to v1a and v1b revisions
Parts:
- gave numbers to parts that had none: 3
- renumbered U24 to U30, U25 to U32
Changed lines of the file:
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@@
   (symbol (lib_id "power:GND") (at 69.85 59.69 270) (unit 1)
     (in_bom yes) (on_board yes) (dnp no) (fields_autoplaced)
-    (property "Reference" "#PWR091" (at 63.5 59.69 0)
+    (property "Reference" "#PWR0130" (at 63.5 59.69 0)
       (effects (font (size 1.27 1.27)) hide)
     )
@@
     (instances
       (project "v1a"
-        (path "/82bc3382-6295-4121-a2db-2433a00f189b"
-          (reference "#PWR091") (unit 1)
-        )
         (path "/82bc3382-6295-4121-a2db-2433a00f189b/610752b3-8dbd-43d5-b875-f3341ea4a837"
           (reference "#PWR0130") (unit 1)
@@
   (symbol (lib_id "power:GND") (at 135.89 96.52 0) (unit 1)
     (in_bom yes) (on_board yes) (dnp no) (fields_autoplaced)
-    (property "Reference" "#PWR0135" (at 135.89 102.87 0)
+    (property "Reference" "#PWR0138" (at 135.89 102.87 0)
       (effects (font (size 1.27 1.27)) hide)
     )
@@
     (instances
       (project "v1a"
-        (path "/82bc3382-6295-4121-a2db-2433a00f189b/0beb40b4-3ea5-423b-b5b9-637bbdbde287"
-          (reference "#PWR0135") (unit 1)
-        )
         (path "/82bc3382-6295-4121-a2db-2433a00f189b/610752b3-8dbd-43d5-b875-f3341ea4a837"
           (reference "#PWR0138") (unit 1)
@@
   (symbol (lib_id "power:+5V") (at 80.01 77.47 270) (unit 1)
     (in_bom yes) (on_board yes) (dnp no) (fields_autoplaced)
-    (property "Reference" "#PWR092" (at 76.2 77.47 0)
+    (property "Reference" "#PWR0134" (at 76.2 77.47 0)
       (effects (font (size 1.27 1.27)) hide)
     )
@@
     (instances
       (project "v1a"
-        (path "/82bc3382-6295-4121-a2db-2433a00f189b"
-          (reference "#PWR092") (unit 1)
-        )
         (path "/82bc3382-6295-4121-a2db-2433a00f189b/610752b3-8dbd-43d5-b875-f3341ea4a837"
           (reference "#PWR0134") (unit 1)
@@
   (symbol (lib_id "power:GND") (at 173.99 76.2 90) (unit 1)
     (in_bom yes) (on_board yes) (dnp no) (fields_autoplaced)
-    (property "Reference" "#PWR0103" (at 180.34 76.2 0)
+    (property "Reference" "#PWR0140" (at 180.34 76.2 0)
       (effects (font (size 1.27 1.27)) hide)
     )
@@
     (instances
       (project "v1a"
-        (path "/82bc3382-6295-4121-a2db-2433a00f189b"
-          (reference "#PWR0103") (unit 1)
-        )
         (path "/82bc3382-6295-4121-a2db-2433a00f189b/610752b3-8dbd-43d5-b875-f3341ea4a837"
           (reference "#PWR0140") (unit 1)
@@
   (symbol (lib_id "power:+5V") (at 173.99 35.56 90) (unit 1)
     (in_bom yes) (on_board yes) (dnp no) (fields_autoplaced)
-    (property "Reference" "#PWR095" (at 177.8 35.56 0)
+    (property "Reference" "#PWR0139" (at 177.8 35.56 0)
       (effects (font (size 1.27 1.27)) hide)
     )
@@
     (instances
       (project "v1a"
-        (path "/82bc3382-6295-4121-a2db-2433a00f189b"
-          (reference "#PWR095") (unit 1)
-        )
         (path "/82bc3382-6295-4121-a2db-2433a00f189b/610752b3-8dbd-43d5-b875-f3341ea4a837"
           (reference "#PWR0139") (unit 1)
@@
   (symbol (lib_id "Device:C") (at 161.29 92.71 0) (unit 1)
     (in_bom yes) (on_board yes) (dnp no) (fields_autoplaced)
-    (property "Reference" "C?" (at 165.1 91.44 0)
+    (property "Reference" "Cd30" (at 165.1 91.44 0)
       (effects (font (size 1.27 1.27)) (justify left))
     )
@@
     (instances
       (project "v1a"
-        (path "/82bc3382-6295-4121-a2db-2433a00f189b/0beb40b4-3ea5-423b-b5b9-637bbdbde287"
-          (reference "C?") (unit 1)
-        )
         (path "/82bc3382-6295-4121-a2db-2433a00f189b/610752b3-8dbd-43d5-b875-f3341ea4a837"
           (reference "Cd30") (unit 1)
@@
   (symbol (lib_id "power:+5V") (at 135.89 88.9 0) (unit 1)
     (in_bom yes) (on_board yes) (dnp no)
-    (property "Reference" "#PWR0136" (at 135.89 92.71 0)
+    (property "Reference" "#PWR0137" (at 135.89 92.71 0)
       (effects (font (size 1.27 1.27)) hide)
     )
@@
     (instances
       (project "v1a"
-        (path "/82bc3382-6295-4121-a2db-2433a00f189b/0beb40b4-3ea5-423b-b5b9-637bbdbde287"
-          (reference "#PWR0136") (unit 1)
-        )
         (path "/82bc3382-6295-4121-a2db-2433a00f189b/610752b3-8dbd-43d5-b875-f3341ea4a837"
           (reference "#PWR0137") (unit 1)
@@
   (symbol (lib_id "Device:C") (at 148.59 92.71 0) (unit 1)
     (in_bom yes) (on_board yes) (dnp no) (fields_autoplaced)
-    (property "Reference" "C?" (at 152.4 91.44 0)
+    (property "Reference" "Cd29" (at 152.4 91.44 0)
       (effects (font (size 1.27 1.27)) (justify left))
     )
@@
     (instances
       (project "v1a"
-        (path "/82bc3382-6295-4121-a2db-2433a00f189b/0beb40b4-3ea5-423b-b5b9-637bbdbde287"
-          (reference "C?") (unit 1)
-        )
         (path "/82bc3382-6295-4121-a2db-2433a00f189b/610752b3-8dbd-43d5-b875-f3341ea4a837"
           (reference "Cd29") (unit 1)
@@
   (symbol (lib_id "74xx:74HC138") (at 80.01 54.61 0) (unit 1)
     (in_bom yes) (on_board yes) (dnp no) (fields_autoplaced)
-    (property "Reference" "U24" (at 82.2041 36.83 0)
+    (property "Reference" "U30" (at 82.2041 36.83 0)
       (effects (font (size 1.27 1.27)) (justify left))
     )
@@
     (instances
       (project "v1a"
-        (path "/82bc3382-6295-4121-a2db-2433a00f189b"
-          (reference "U24") (unit 1)
-        )
         (path "/82bc3382-6295-4121-a2db-2433a00f189b/610752b3-8dbd-43d5-b875-f3341ea4a837"
           (reference "U30") (unit 1)
@@
   (symbol (lib_id "power:GND") (at 80.01 67.31 90) (unit 1)
     (in_bom yes) (on_board yes) (dnp no) (fields_autoplaced)
-    (property "Reference" "#PWR089" (at 86.36 67.31 0)
+    (property "Reference" "#PWR0133" (at 86.36 67.31 0)
       (effects (font (size 1.27 1.27)) hide)
     )
@@
     (instances
       (project "v1a"
-        (path "/82bc3382-6295-4121-a2db-2433a00f189b"
-          (reference "#PWR089") (unit 1)
-        )
         (path "/82bc3382-6295-4121-a2db-2433a00f189b/610752b3-8dbd-43d5-b875-f3341ea4a837"
           (reference "#PWR0133") (unit 1)
@@
   (symbol (lib_id "74xx:74AHC273") (at 173.99 55.88 0) (unit 1)
     (in_bom yes) (on_board yes) (dnp no) (fields_autoplaced)
-    (property "Reference" "U25" (at 176.1841 35.56 0)
+    (property "Reference" "U32" (at 176.1841 35.56 0)
       (effects (font (size 1.27 1.27)) (justify left))
     )
@@
     (instances
       (project "v1a"
-        (path "/82bc3382-6295-4121-a2db-2433a00f189b"
-          (reference "U25") (unit 1)
-        )
         (path "/82bc3382-6295-4121-a2db-2433a00f189b/610752b3-8dbd-43d5-b875-f3341ea4a837"
           (reference "U32") (unit 1)
@@
   (symbol (lib_id "power:GND") (at 125.73 74.93 90) (unit 1)
     (in_bom yes) (on_board yes) (dnp no) (fields_autoplaced)
-    (property "Reference" "#PWR094" (at 132.08 74.93 0)
+    (property "Reference" "#PWR0136" (at 132.08 74.93 0)
       (effects (font (size 1.27 1.27)) hide)
     )
@@
     (instances
       (project "v1a"
-        (path "/82bc3382-6295-4121-a2db-2433a00f189b"
-          (reference "#PWR094") (unit 1)
-        )
         (path "/82bc3382-6295-4121-a2db-2433a00f189b/610752b3-8dbd-43d5-b875-f3341ea4a837"
           (reference "#PWR0136") (unit 1)
@@
   (symbol (lib_id "Device:C") (at 135.89 92.71 0) (unit 1)
     (in_bom yes) (on_board yes) (dnp no) (fields_autoplaced)
-    (property "Reference" "C?" (at 139.7 91.44 0)
+    (property "Reference" "Cd28" (at 139.7 91.44 0)
       (effects (font (size 1.27 1.27)) (justify left))
     )
@@
     (instances
       (project "v1a"
-        (path "/82bc3382-6295-4121-a2db-2433a00f189b/0beb40b4-3ea5-423b-b5b9-637bbdbde287"
-          (reference "C?") (unit 1)
-        )
         (path "/82bc3382-6295-4121-a2db-2433a00f189b/610752b3-8dbd-43d5-b875-f3341ea4a837"
           (reference "Cd28") (unit 1)
@@
   (symbol (lib_id "power:+5V") (at 80.01 36.83 90) (unit 1)
     (in_bom yes) (on_board yes) (dnp no) (fields_autoplaced)
-    (property "Reference" "#PWR090" (at 83.82 36.83 0)
+    (property "Reference" "#PWR0132" (at 83.82 36.83 0)
       (effects (font (size 1.27 1.27)) hide)
     )
@@
     (instances
       (project "v1a"
-        (path "/82bc3382-6295-4121-a2db-2433a00f189b"
-          (reference "#PWR090") (unit 1)
-        )
         (path "/82bc3382-6295-4121-a2db-2433a00f189b/610752b3-8dbd-43d5-b875-f3341ea4a837"
           (reference "#PWR0132") (unit 1)
@@
   (symbol (lib_id "power:+5V") (at 125.73 34.29 90) (unit 1)
     (in_bom yes) (on_board yes) (dnp no) (fields_autoplaced)
-    (property "Reference" "#PWR093" (at 129.54 34.29 0)
+    (property "Reference" "#PWR0135" (at 129.54 34.29 0)
       (effects (font (size 1.27 1.27)) hide)
     )
@@
     (instances
       (project "v1a"
-        (path "/82bc3382-6295-4121-a2db-2433a00f189b"
-          (reference "#PWR093") (unit 1)
-        )
         (path "/82bc3382-6295-4121-a2db-2433a00f189b/610752b3-8dbd-43d5-b875-f3341ea4a837"
           (reference "#PWR0135") (unit 1)
