File: Kicad/v1a/memory.kicad_sch (KiCad schematic)
At the start: 11 parts, among them U21 62256, U29 SST39SF, U7 74HC00, U8 74HC85

Commit message: Add files relating to v1a and v1b revisions
Parts:
- gave numbers to parts that had none: 4
- renumbered D1 to D4, D1 to D5, R1 to R37, U7 to U26, U8 to U27, U21 to U28
