File: Kicad/v1a/ports.kicad_sch (KiCad schematic)
At the start: 14 parts, among them J1 Barrel_Jack_MountingPin, J2 SCART-F, J5 Conn_02x22_Odd_Even, J6 Conn_02x22_Odd_Even, SW1 SW_DPDT_x2

Commit message: Add files relating to v1a and v1b revisions
Parts:
- renumbered J1 to J3, J2 to J4, SW1 to SW2
Other:
- note added: "Bottom Side"
- note added: "Top Side"
- moved on the sheet: C7, C8, J6
