File: Kicad/v1a/v1a.kicad_sch (KiCad schematic)
At the start: 11 parts, among them U1 65c02

Commit message: Add files relating to v1a and v1b revisions
Parts:
- gave numbers to parts that had none: 1
Changed lines of the file:
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@@
   (symbol (lib_id "Device:C") (at 87.63 66.04 0) (unit 1)
     (in_bom yes) (on_board yes) (dnp no) (fields_autoplaced)
-    (property "Reference" "C?" (at 91.44 64.77 0)
+    (property "Reference" "Cd1" (at 91.44 64.77 0)
       (effects (font (size 1.27 1.27)) (justify left))
     )
@@
     (instances
       (project "v1a"
-        (path "/82bc3382-6295-4121-a2db-2433a00f189b/0beb40b4-3ea5-423b-b5b9-637bbdbde287"
-          (reference "C?") (unit 1)
-        )
         (path "/82bc3382-6295-4121-a2db-2433a00f189b"
           (reference "Cd1") (unit 1)
@@
   (symbol (lib_id "power:GND") (at 87.63 69.85 0) (unit 1)
     (in_bom yes) (on_board yes) (dnp no)
-    (property "Reference" "#PWR0135" (at 87.63 76.2 0)
+    (property "Reference" "#PWR05" (at 87.63 76.2 0)
       (effects (font (size 1.27 1.27)) hide)
     )
@@
     (instances
       (project "v1a"
-        (path "/82bc3382-6295-4121-a2db-2433a00f189b/0beb40b4-3ea5-423b-b5b9-637bbdbde287"
-          (reference "#PWR0135") (unit 1)
-        )
         (path "/82bc3382-6295-4121-a2db-2433a00f189b"
           (reference "#PWR05") (unit 1)
@@
   (symbol (lib_id "power:+5V") (at 87.63 62.23 0) (unit 1)
     (in_bom yes) (on_board yes) (dnp no)
-    (property "Reference" "#PWR0136" (at 87.63 66.04 0)
+    (property "Reference" "#PWR04" (at 87.63 66.04 0)
       (effects (font (size 1.27 1.27)) hide)
     )
@@
     (instances
       (project "v1a"
-        (path "/82bc3382-6295-4121-a2db-2433a00f189b/0beb40b4-3ea5-423b-b5b9-637bbdbde287"
-          (reference "#PWR0136") (unit 1)
-        )
         (path "/82bc3382-6295-4121-a2db-2433a00f189b"
           (reference "#PWR04") (unit 1)
